File: Hardware/Led_Control.sch (KiCad schematic (older format))
At the start: 17 parts, among them Q2 BC848, Q3 BC848, Q4 BC848, Q5 BC848, Q6 BC848, Q7 BC848, Q8 BC848, Q9 BCX51,115

Commit message: Added the ring counter to the schematic.
Parts:
- Q9: value BCX51,115 -> BCX51; ManufacturerPartNumber (none) -> BCX51,115
Connections:
- net +5V: now also R3.2
- net GND: no longer R3.2
Changed lines of the file:
@@
 $Descr A4 11693 8268
 encoding utf-8
-Sheet 2 2
+Sheet 2 3
 Title "Leds control logic and power"
-Date ""
+Date "2022-01-01"
 Rev ""
 Comp "(C) Adrien RICCIARDI"
@@
 P 7550 2250
 F 0 "Q9" H 7740 2204 50  0000 L CNN
-F 1 "BCX51,115" H 7740 2295 50  0000 L CNN
+F 1 "BCX51" H 7740 2295 50  0000 L CNN
 F 2 "Package_TO_SOT_SMD:SOT-89-3" H 7750 2175 50  0001 L CIN
 F 3 "http://www.infineon.com/dgdl/bcx51_bcx52_bcx53.pdf" H 7550 2250 50  0001 L CNN
@@
 F 7 "Spice_Simulation/BCX51.lib" H 7550 2250 50  0001 C CNN "Spice_Lib_File"
 F 8 "3 1 2" H 7550 2250 50  0001 C CNN "Spice_Node_Sequence"
+F 9 "BCX51,115" H 7550 2250 50  0001 C CNN "ManufacturerPartNumber"
 	1    7550 2250
 	1    0    0    1
@@
 P 2100 5000
 AR Path="/61D82050" Ref="#PWR?"  Part="1"
-AR Path="/61CE6682/61D82050" Ref="#PWR?"  Part="1"
-F 0 "#PWR?" H 2100 4750 50  0001 C CNN
+AR Path="/61CE6682/61D82050" Ref="#PWR08"  Part="1"
+F 0 "#PWR08" H 2100 4750 50  0001 C CNN
 F 1 "GND" H 2105 4827 50  0000 C CNN
 F 2 "" H 2100 5000 50  0001 C CNN
@@
 $EndComp
 $Comp
-L power:GND #PWR?
-U 1 1 61D82878
+L power:+5V #PWR?
+U 1 1 61FED532
 P 2100 3350
-AR Path="/61D82878" Ref="#PWR?"  Part="1"
-AR Path="/61CE6682/61D82878" Ref="#PWR?"  Part="1"
-F 0 "#PWR?" H 2100 3100 50  0001 C CNN
-F 1 "GND" H 2105 3177 50  0000 C CNN
+AR Path="/61FED532" Ref="#PWR?"  Part="1"
+AR Path="/61CE6682/61FED532" Ref="#PWR?"  Part="1"
+F 0 "#PWR?" H 2100 3200 50  0001 C CNN
+F 1 "+5V" H 2115 3523 50  0000 C CNN
 F 2 "" H 2100 3350 50  0001 C CNN
 F 3 "" H 2100 3350 50  0001 C CNN
+F 4 "V" H 2100 3350 50  0001 C CNN "Spice_Primitive"
+F 5 "dc 5" H 2100 3350 50  0001 C CNN "Spice_Model"
+F 6 "Y" H 2100 3350 50  0001 C CNN "Spice_Netlist_Enabled"
 	1    2100 3350
-	1    0    0    -1
+	-1   0    0    1
 $EndComp
 $EndSCHEMATC

Commit message: Improved ring counter RS latches output with better signal quality and less transistors count.
Parts:
- added R?: 1K, Resistor_SMD:R_0603_1608Metric_Pad0.98x0.95mm_HandSolder, symbol Device:R
Connections:
- net +5V: no longer R3.2
- net GND: no longer Q8.1 (B), R4.2
- new net: Q8.1 (B), R?.2
- new net COUNTER_BIT_0: R3.2
- new net COUNTER_BIT_1: R4.2, R?.1
Changed lines of the file:
@@
 	4150 2100 4500 2100
 Wire Wire Line
-	2100 3350 2100 3250
-Wire Wire Line
 	2100 3250 2200 3250
-Wire Wire Line
-	2100 5000 2100 4950
-Wire Wire Line
-	2100 4850 2200 4850
 Wire Notes Line
 	2600 5550 3300 5550
@@
 Wire Wire Line
 	5900 2500 5850 2500
-Wire Wire Line
-	5850 2500 5850 5650
 $Comp
 L Device:R R?
@@
 Wire Wire Line
 	8600 2950 8600 3050
-Text Notes 1800 3450 0    50   Italic 10
-TEST
-Text Notes 1800 5000 0    50   Italic 10
-TEST
 Text Notes 8300 2850 0    50   Italic 10
 TEST
 Wire Wire Line
-	2100 4950 2400 4950
-Wire Wire Line
-	2400 4950 2400 5650
-Connection ~ 2100 4950
-Wire Wire Line
-	2100 4950 2100 4850
-Wire Wire Line
 	2500 4850 2600 4850
 Wire Wire Line
-	2400 5650 5850 5650
-$Comp
-L power:GND #PWR?
-U 1 1 61D82050
-P 2100 5000
-AR Path="/61D82050" Ref="#PWR?"  Part="1"
-AR Path="/61CE6682/61D82050" Ref="#PWR08"  Part="1"
-F 0 "#PWR08" H 2100 4750 50  0001 C CNN
-F 1 "GND" H 2105 4827 50  0000 C CNN
-F 2 "" H 2100 5000 50  0001 C CNN
-F 3 "" H 2100 5000 50  0001 C CNN
-	1    2100 5000
-	1    0    0    -1
-$EndComp
-$Comp
-L power:+5V #PWR?
-U 1 1 61FED532
-P 2100 3350
-AR Path="/61FED532" Ref="#PWR?"  Part="1"
-AR Path="/61CE6682/61FED532" Ref="#PWR?"  Part="1"
-F 0 "#PWR?" H 2100 3200 50  0001 C CNN
-F 1 "+5V" H 2115 3523 50  0000 C CNN
-F 2 "" H 2100 3350 50  0001 C CNN
-F 3 "" H 2100 3350 50  0001 C CNN
-F 4 "V" H 2100 3350 50  0001 C CNN "Spice_Primitive"
-F 5 "dc 5" H 2100 3350 50  0001 C CNN "Spice_Model"
-F 6 "Y" H 2100 3350 50  0001 C CNN "Spice_Netlist_Enabled"
-	1    2100 3350
+	5850 2500 5850 2700
+Wire Wire Line
+	2150 5700 5850 5700
+$Comp
+L Device:R R?
+U 1 1 62BA8E39
+P 5850 2850
+AR Path="/62BA8E39" Ref="R?"  Part="1"
+AR Path="/61CE6682/62BA8E39" Ref="R?"  Part="1"
+F 0 "R?" H 5919 2759 50  0000 L CNN
+F 1 "1K" H 5919 2850 50  0000 L CNN
+F 2 "Resistor_SMD:R_0603_1608Metric_Pad0.98x0.95mm_HandSolder" V 5780 2850 50  0001 C CNN
+F 3 "~" H 5850 2850 50  0001 C CNN
+F 4 "5%" H 5919 2941 50  0000 L CNN "Value2"
+F 5 "R" H 5850 2850 50  0001 C CNN "Spice_Primitive"
+F 6 "1k" H 5850 2850 50  0001 C CNN "Spice_Model"
+F 7 "Y" H 5850 2850 50  0001 C CNN "Spice_Netlist_Enabled"
+	1    5850 2850
 	-1   0    0    1
 $EndComp
+Wire Wire Line
+	5850 3000 5850 5700
+Text HLabel 2100 3250 0    50   Input ~ 0
+COUNTER_BIT_0
+Text HLabel 2100 4850 0    50   Input ~ 0
+COUNTER_BIT_1
+Connection ~ 2150 4850
+Wire Wire Line
+	2150 4850 2200 4850
+Wire Wire Line
+	2100 4850 2150 4850
+Wire Wire Line
+	2150 4850 2150 5700
 $EndSCHEMATC

Commit message: Added second led logic and power transistor, also added BC858 SPICE model.
Parts:
- added Q44: BC848, Package_TO_SOT_SMD:SOT-23, symbol Transistor_BJT:BC848
- added Q45: BCX51, Package_TO_SOT_SMD:SOT-89-3, symbol Transistor_BJT:BCX51
- added R66, R67, R69: 1K, Resistor_SMD:R_0603_1608Metric_Pad0.98x0.95mm_HandSolder, symbol Device:R
- added R68: 560, Resistor_SMD:R_0603_1608Metric_Pad0.98x0.95mm_HandSolder, symbol Device:R
- gave numbers to parts that had none: 1
Connections:
- net +5V: now also Q45.3 (E), R67.2
- net COUNTER_BIT_0: now also R66.2
- net GND: now also Q44.2 (E), R69.2
- new net: Q44.1 (B), R66.1
- new net: Q44.3 (C), R67.1, R68.2
- new net: Q45.2 (C), R69.1
- new net: Q45.1 (B), R68.1

Commit message: Added RS latches power-on reset.
Parts:
- Q45, Q9: ManufacturerPartNumber BCX51,115 -> (none); PartNumber (none) -> BCX51,115
Changed lines of the file:
@@
 F 7 "Spice_Simulation/BCX51.lib" H 7550 2250 50  0001 C CNN "Spice_Lib_File"
 F 8 "3 1 2" H 7550 2250 50  0001 C CNN "Spice_Node_Sequence"
-F 9 "BCX51,115" H 7550 2250 50  0001 C CNN "ManufacturerPartNumber"
+F 9 "BCX51,115" H 7550 2250 50  0001 C CNN "PartNumber"
 	1    7550 2250
 	1    0    0    1
@@
 F 7 "Spice_Simulation/BCX51.lib" H 8800 4550 50  0001 C CNN "Spice_Lib_File"
 F 8 "3 1 2" H 8800 4550 50  0001 C CNN "Spice_Node_Sequence"
-F 9 "BCX51,115" H 8800 4550 50  0001 C CNN "ManufacturerPartNumber"
+F 9 "BCX51,115" H 8800 4550 50  0001 C CNN "PartNumber"
 	1    8800 4550
 	1    0    0    1

Commit message: Added oscillator to schematic.
Other:
- note added: "Power PNP transistors base resistor value :\n\nLet's decide that maximum emitter current will be 500 mA\n(enough for 30 leds at 15 mA each).\nMinimum hFE is 63. So minimum base current is 0.5A / 63hFE = 8 mA.\nAs R = U / I, the maximum base resistor value is\n5V / 0.008A = 625 ohm.\nUse a 560 ohm resistor to get a little more margin."
- note removed: "PNP transistors base resistor value :\n\nLet's decide that maximum emitter current will be 500 mA\n(enough for 30 leds at 15 mA each).\nMinimum hFE is 63. So minimum base current is 0.5A / 63hFE = 8 mA.\nAs R = U / I, the maximum base resistor value is\n5V / 0.008A = 625 ohm.\nUse a 560 ohm resistor to get a little more margin."
Changed lines of the file:
@@
 $Descr A4 11693 8268
 encoding utf-8
-Sheet 2 3
+Sheet 2 4
 Title "Leds control logic and power"
 Date "2022-01-01"
@@
 $EndComp
 Text Notes 2900 7350 0    50   ~ 0
-PNP transistors base resistor value :\n\nLet's decide that maximum emitter current will be 500 mA\n(enough for 30 leds at 15 mA each).\nMinimum hFE is 63. So minimum base current is 0.5A / 63hFE = 8 mA.\nAs R = U / I, the maximum base resistor value is\n5V / 0.008A = 625 ohm.\nUse a 560 ohm resistor to get a little more margin.
+Power PNP transistors base resistor value :\n\nLet's decide that maximum emitter current will be 500 mA\n(enough for 30 leds at 15 mA each).\nMinimum hFE is 63. So minimum base current is 0.5A / 63hFE = 8 mA.\nAs R = U / I, the maximum base resistor value is\n5V / 0.008A = 625 ohm.\nUse a 560 ohm resistor to get a little more margin.
 Connection ~ 6200 2250
 Wire Wire Line
