File: Motherboard/Hardware/Ring_Counter.kicad_sch (KiCad schematic)
At the start: 89 parts, among them Q11 BC848, Q12 BC858, Q13 BC858, Q14 BC858, Q15 BC858, Q16 BC858, Q17 BC858, Q18 BC848, Q19 BC848, Q20 BC848, Q21 BC848, Q22 BC848, Q23 BC848, Q24 BC848, Q25 BC848, Q26 BC848, Q27 BC848, Q28 BC848, Q29 BC848, Q30 BC858, Q31 BC848, Q32 BC858, Q33 BC858, Q34 BC858, Q35 BC858, Q36 BC858, Q37 BC848, Q38 BC848, Q39 BC848, Q40 BC848, Q41 BC848, Q42 BC848, Q43 BC848, Q44 BC848, Q45 BC858

Commit message: Updated the motherboard PCB to KiCad 7.
Parts:
- Q11, Q18, Q19, Q20, Q21, Q22, Q23, Q24, Q25, Q26, Q27, Q28, Q29, Q31, Q37, Q38, Q39, Q40, Q41, Q42, Q43, Q44: Spice_Lib_File Spice_Simulation/BC848.lib -> (none); Spice_Model BC848 -> (none); Spice_Netlist_Enabled Y -> (none); Spice_Node_Sequence 3 1 2 -> (none); Spice_Primitive Q -> (none)
- Q12, Q13, Q14, Q15, Q16, Q17, Q30, Q32, Q33, Q34, Q35, Q36, Q45: Spice_Lib_File Spice_Simulation/BC858.lib -> (none); Spice_Model BC858 -> (none); Spice_Netlist_Enabled Y -> (none); Spice_Node_Sequence 3 1 2 -> (none); Spice_Primitive Q -> (none)
- R13, R14, R18, R19, R20, R21, R22, R23, R33, R34, R35, R43, R44, R45, R50, R51, R52, R53, R60, R61, R67, R74: Spice_Model 1k -> (none); Spice_Netlist_Enabled Y -> (none); Spice_Primitive R -> (none)
- R15, R16, R17, R24, R25, R26, R27, R28, R29, R30, R31, R32, R36, R37, R38, R39, R40, R41, R42, R48, R49, R54, R55, R56, R57, R58, R59, R62, R63, R64, R65, R66: Spice_Model 10k -> (none); Spice_Netlist_Enabled Y -> (none); Spice_Primitive R -> (none)
